Commit message: feat(robot): UR5e-shaped skeleton + seed TCP at the flange, not the base
Two fixes to the robot display:

1) TCP no longer overlaps the base. `ROBOT_FRAME_DEFAULTS[tcp]` was a dead
   constant — ensureRobotFrames created the tcp child frame at local (0,0,0),
   coincident with robot_base. The tool point now seeds at the skeleton's
   flange (tool0) instead: its default LOCAL translation is the forward
   kinematics of RobotStage's rest pose, base-frame (-0.717,-0.133,0.346),
   and ensureRobotFrames applies it to the newly-created frame. Orientation
   stays identity so the grasp-search wire contract (tcpOrientation) is
   unchanged until the user re-aims it.

2) Skeleton is now UR-shaped. Replaced the coaxial "totem pole" URDF with one
   whose joint origins reproduce the Universal Robots UR5e link transforms
   (d1/a2/a3/d4/d5/d6), giving the recognizable UR silhouette — the two offset
   arm links + the three-axis wrist cluster. Still self-contained: primitive
   cylinder "bone + knuckle" geometry, no external mesh assets (GitHub-Pages
   friendly, no `packages` mapping). Joint names keep the UR convention so
   RobotStage._applyRestPose and any grasp-contract joint payload still key
   against them.

Rest pose (RobotStage._applyRestPose) and the tcp seed are a coupled pair,
documented in both files. Verified: urdf-loader renders the flange at exactly
the seeded value; full JS suite (701) green; production build clean.

Co-Authored-By: Claude Opus 4.8 <noreply@anthropic.com>
Claude-Session: https://claude.ai/code/session_01BYJ8QG6njDHRVCXo4SWe57

File: public/robot/skeleton_arm.urdf (robot description, URDF)
Before this commit: robot skeleton_arm, 7 links, 6 joints
Links:
- removed link flange
- added link wrist_3_link; visual cylinder length=0.02 radius=0.031; visual cylinder length=0.05 radius=0.038
- link base_link: geometry visual cylinder length=0.163 radius=0.075
- link forearm_link: geometry visual cylinder length=0.11 radius=0.046; visual cylinder length=0.1333 radius=0.038
- link shoulder_link: geometry visual cylinder length=0.14 radius=0.062
- link upper_arm_link: geometry visual cylinder length=0.13 radius=0.058; visual cylinder length=0.425 radius=0.05
- link wrist_1_link: geometry visual cylinder length=0.09 radius=0.042; visual cylinder length=0.0997 radius=0.038
- link wrist_2_link: geometry visual cylinder length=0.085 radius=0.04; visual cylinder length=0.0996 radius=0.036
Joints:
- joint elbow_joint: axis 0 1 0 -> 0 0 1; limit lower=-2.618 upper=2.618 effort=100 velocity=3.14 -> lower=-3.1416 upper=3.1416 effort=150 velocity=3.14; origin xyz=0 0 0.30 rpy=0 0 0 -> xyz=-0.425 0 0 rpy=0 0 0
- joint shoulder_lift_joint: axis 0 1 0 -> 0 0 1; limit lower=-2.0944 upper=2.0944 effort=150 velocity=3.14 -> lower=-6.2832 upper=6.2832 effort=150 velocity=3.14; origin xyz=0 0 0.12 rpy=0 0 0 -> xyz=0 0 0 rpy=1.570796327 0 0
- joint shoulder_pan_joint: limit lower=-2.967 upper=2.967 effort=150 velocity=3.14 -> lower=-6.2832 upper=6.2832 effort=150 velocity=3.14; origin xyz=0 0 0.08 rpy=0 0 0 -> xyz=0 0 0.1625 rpy=0 0 0
- joint wrist_1_joint: axis 0 1 0 -> 0 0 1; limit lower=-3.14159 upper=3.14159 effort=30 velocity=6.28 -> lower=-6.2832 upper=6.2832 effort=28 velocity=6.28; origin xyz=0 0 0.25 rpy=0 0 0 -> xyz=-0.3922 0 0.1333 rpy=0 0 0
- joint wrist_2_joint: axis 1 0 0 -> 0 0 1; limit lower=-3.14159 upper=3.14159 effort=30 velocity=6.28 -> lower=-6.2832 upper=6.2832 effort=28 velocity=6.28; origin xyz=0 0 0.08 rpy=0 0 0 -> xyz=0 -0.0997 0 rpy=1.570796327 0 0
- joint wrist_3_joint: child flange -> wrist_3_link; limit lower=-3.14159 upper=3.14159 effort=30 velocity=6.28 -> lower=-6.2832 upper=6.2832 effort=28 velocity=6.28; origin xyz=0 0 0.06 rpy=0 0 0 -> xyz=0 0.0996 0 rpy=1.570796327 3.141592654 3.141592654

Commit message: fix(robot): ツールはフランジに固定され、腕は一度だけ現れる (ADR-150)
当事者の /whiteboard 依頼 3 点への対応。

- スポーン時のちらつき: 実写メッシュを 1 つの共有資産 (idle/loading/ready/
  failed) にし、stage は clone、起動時に先読み。宣言スタイルが着地するまで
  腕を隠し、RobotAppearanceToggle の固定スロットに LOADING… を出す。失敗
  したら skeleton を見せて toast (不可視のまま残さない)。
- 関節構造の見た目: skeleton_arm.urdf の visual だけを UR メッシュの骨の
  平面 (上腕 z=0.138 / 前腕 z=0.007) へ。関節原点は不変。
- ツール: robot.toolLength (request 側 optional、contractVersion=6 据え置き)。
  core/ はフランジを TCP から approach の逆向きに戻して解き、フランジ→TCP
  区間を干渉判定にかける。front は常に 150mm を宣言し、wrist_3_link の子と
  してツールを描く。腕が候補を持つときゴーストはハンドを描かない。
- 実装中に発見: 平行ジョーの閉じ軸がフランジ座標で roll の 2 倍で回って
  いた (ADR-147 の gauge がフランジ x を張り直していた)。候補 frame の x 軸
  まわり 180° の固定取付けに正した。代表解の枝が変わり、ペデスタル受け入れ
  値は 10 → 4。

残し: DEF-043 (単体/トレー内ピック検証の分割 — 別 PR)、DEF-044 (tcp
フレームの seed はフランジ位置のまま)。

Co-Authored-By: Claude Opus 5.5 <noreply@anthropic.com>
Claude-Session: https://claude.ai/code/session_01WJQniUwHTFx1oqyjTNfKvT
Model-Effort: claude-opus-5-5/medium
Task-Class: fix/bff+build+contract+core+docs+front+governance

File: public/robot/skeleton_arm.urdf (robot description, URDF)
Before this commit: robot ur5e_skeleton, 7 links, 6 joints
Links:
- link forearm_link: geometry visual cylinder length=0.1263 radius=0.038; visual cylinder length=0.225 radius=0.046
- link upper_arm_link: geometry visual cylinder length=0.21 radius=0.058; visual cylinder length=0.425 radius=0.05
